File: KiCAD/Main Board/Main Board.kicad_pcb (KiCad board)
At the start: 2 copper layers, 65 x 56 mm, 12 parts, among them J1 Conn_02x10_Odd_Even, J2 ATtiny84 I2C/SPI Debug, J3 ATtiny85 I2c/SPI Debug, P1 Raspberry Pi, U1 ATtiny84-20PU, U2 ATtiny85-20PU

Commit message: OSHPARK Order Number chh9sp7Z
Signed-off-by: John Jacques <eruditelite@gmail.com>
Parts:
- J1: value Conn_02x10_Odd_Even -> Daughter Board Connector
Connections:
- P1 pad 2: +5V -> Net-(P1-Pad2)
- P1 pad 34: GND -> Net-(P1-Pad34)
- P1 pad 6: GND -> Net-(P1-Pad6)
- P1 pad 9: GND -> Net-(P1-Pad9)
Routing:
- net GND: track 119.1 -> 33.8 mm, vias 2 -> 1
- net +5V: track 37.1 -> 34.6 mm
- net /GPIO11(SPI0_SCK): track 79.5 -> 80.2 mm
Other:
- board text added: "ATTiny Examples eruditelite@gmail.com"
- board text added: "Clock"
- board text added: "MISO"
- board text added: "SDA/MOSI"
