File: KiCAD/Main Board/Main Board.sch (KiCad schematic (older format))
At the start: 12 parts, among them J1 Daughter Board Connector, J2 ATtiny84 I2C/SPI Debug, J3 ATtiny85 I2c/SPI Debug, P1 Raspberry Pi, U1 ATtiny84-20PU, U2 ATtiny85-20PU

Commit message: OSHPARK Order Number chh9sp7Z
Signed-off-by: John Jacques <eruditelite@gmail.com>
Connections:
- net +5V: no longer P1.2 (Pin_2)
- net GND: no longer P1.34 (Pin_34), P1.6 (Pin_6), P1.9 (Pin_9)
- no-connect marks 21 -> 25
Changed lines of the file:
@@
 $EndComp
-Wire Wire Line
-	2450 2700 2450 2850
-Wire Wire Line
-	2450 2850 2650 2850
 Wire Wire Line
 	2450 2950 2650 2950
-Connection ~ 2450 2850
-$Comp
-L power:GND #PWR02
-U 1 1 580C1D11
-P 2550 4900
-F 0 "#PWR02" H 2550 4650 50  0001 C CNN
-F 1 "GND" H 2550 4750 50  0000 C CNN
-F 2 "" H 2550 4900 50  0000 C CNN
-F 3 "" H 2550 4900 50  0000 C CNN
-	1    2550 4900
-	-1   0    0    -1
-$EndComp
 $Comp
 L power:GND #PWR03
@@
 	-1   0    0    -1
 $EndComp
-Wire Wire Line
-	3250 3250 3150 3250
 Wire Wire Line
 	4300 3150 3150 3150
@@
 Text Label 1600 3250 0    50   ~ 0
 GPIO15(RXD0)
-Wire Wire Line
-	2550 3050 2650 3050
 Text Notes 650  7600 0    50   ~ 0
 ID_SD and ID_SC PINS:\nThese pins are reserved for HAT ID EEPROM.\n\nAt boot time this I2C interface will be\ninterrogated to look for an EEPROM\nthat identifes the attached board and\nallows automagic setup of the GPIOs\n(and optionally, Linux drivers).\n\nDO NOT USE these pins for anything other\nthan attaching an I2C ID EEPROM. Leave\nunconnected if ID EEPROM not required.
@@
 Text Label 1600 4750 0    50   ~ 0
 GPIO21(SPI1_SCK)
-Wire Wire Line
-	2450 2850 2450 2950
 Wire Wire Line
 	3350 2850 3350 3650
@@
 NoConn ~ 2650 3750
 NoConn ~ 2650 3450
-Wire Wire Line
-	3250 3250 3250 4750
-Wire Wire Line
-	2550 3050 2550 4450
 $Comp
 L power:+3.3V #PWR0101
@@
 	10000 3000 11000 3000
 Wire Wire Line
-	2650 4450 2550 4450
-Connection ~ 2550 4450
-Wire Wire Line
-	2550 4450 2550 4900
-Wire Wire Line
 	3150 4750 3250 4750
-Connection ~ 3250 4750
 Wire Wire Line
 	3250 4750 3250 4900
+NoConn ~ 2650 3050
+NoConn ~ 3150 3250
+NoConn ~ 2650 4450
+NoConn ~ 2650 2850
+Wire Wire Line
+	2450 2700 2450 2950
 $EndSCHEMATC
