File: KiCAD/Expansion Boards/Blink/Blink.kicad_pcb (KiCad board)
At the start: 2 copper layers, 29 x 46 mm, 13 parts, among them J1 Daughter Board Connector

Commit message: Ordered Three Blink Boards
OSHPARK order number is XsFSM6ru.

Signed-off-by: John Jacques <eruditelite@gmail.com>
Parts:
- moved D5 0.50 mm to (159.0, 64.5)
Other:
- board text added: "BLIINK"
- board text added: "PB0@84"
- board text added: "PB0@85"
- board text added: "PB1@84"
- board text added: "PB1@85"
- board text added: "PB2@84"
- board text added: "PB2@85"
Changed lines of the file:
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@@
   (general
     (thickness 1.6)
-    (drawings 4)
+    (drawings 11)
     (tracks 67)
     (zones 0)
@@
     (descr "LED, diameter 3.0mm z-position of LED center 2.0mm, 2 pins")
     (tags "LED diameter 3.0mm z-position of LED center 2.0mm 2 pins")
-    (fp_text reference D1 (at 1.27 1.96) (layer B.SilkS)
+    (fp_text reference D1 (at 1.27 1.96) (layer B.SilkS) hide
       (effects (font (size 1 1) (thickness 0.15)) (justify mirror))
     )
@@
     (descr "LED, diameter 3.0mm z-position of LED center 2.0mm, 2 pins")
     (tags "LED diameter 3.0mm z-position of LED center 2.0mm 2 pins")
-    (fp_text reference D2 (at 1.27 1.96) (layer B.SilkS)
+    (fp_text reference D2 (at 1.27 1.96) (layer B.SilkS) hide
       (effects (font (size 1 1) (thickness 0.15)) (justify mirror))
     )
@@
     (descr "LED, diameter 3.0mm z-position of LED center 2.0mm, 2 pins")
     (tags "LED diameter 3.0mm z-position of LED center 2.0mm 2 pins")
-    (fp_text reference D3 (at 1.27 1.96) (layer B.SilkS)
+    (fp_text reference D3 (at 1.27 1.96) (layer B.SilkS) hide
       (effects (font (size 1 1) (thickness 0.15)) (justify mirror))
     )
@@
     (descr "LED, diameter 3.0mm z-position of LED center 2.0mm, 2 pins")
     (tags "LED diameter 3.0mm z-position of LED center 2.0mm 2 pins")
-    (fp_text reference D4 (at 1.27 1.96) (layer B.SilkS)
+    (fp_text reference D4 (at 1.27 1.96) (layer B.SilkS) hide
       (effects (font (size 1 1) (thickness 0.15)) (justify mirror))
     )
@@
   )
   (module LED_THT:LED_D3.0mm_Horizontal_O1.27mm_Z2.0mm (layer B.Cu)
-    (at 159 65)
+    (at 159 64.5)
     (descr "LED, diameter 3.0mm z-position of LED center 2.0mm, 2 pins")
     (tags "LED diameter 3.0mm z-position of LED center 2.0mm 2 pins")
-    (fp_text reference D5 (at 1.27 1.96) (layer B.SilkS)
+    (fp_text reference D5 (at 1.27 1.96) (layer B.SilkS) hide
       (effects (font (size 1 1) (thickness 0.15)) (justify mirror))
     )
@@
     (descr "LED, diameter 3.0mm z-position of LED center 2.0mm, 2 pins")
     (tags "LED diameter 3.0mm z-position of LED center 2.0mm 2 pins")
-    (fp_text reference D6 (at 1.27 1.96) (layer B.SilkS)
+    (fp_text reference D6 (at 1.27 1.96) (layer B.SilkS) hide
       (effects (font (size 1 1) (thickness 0.15)) (justify mirror))
     )
@@
     )
   )
+  (gr_text BLIINK (at 140 46.5 90) (layer B.SilkS)
+    (effects (font (size 1.5 1.5) (thickness 0.3)) (justify mirror))
+  )
+  (gr_text PB2@84 (at 150.5 84) (layer B.SilkS)
+    (effects (font (size 1 1) (thickness 0.1)) (justify mirror))
+  )
+  (gr_text PB2@85 (at 160 84) (layer B.SilkS)
+    (effects (font (size 1 1) (thickness 0.1)) (justify mirror))
+  )
+  (gr_text PB1@85 (at 160 67.5) (layer B.SilkS)
+    (effects (font (size 1 1) (thickness 0.1)) (justify mirror))
+  )
+  (gr_text PB1@84 (at 150.5 67.5) (layer B.SilkS)
+    (effects (font (size 1 1) (thickness 0.1)) (justify mirror))
+  )
+  (gr_text PB0@85 (at 160 52) (layer B.SilkS)
+    (effects (font (size 1 1) (thickness 0.1)) (justify mirror))
+  )
+  (gr_text PB0@84 (at 150.5 52) (layer B.SilkS)
+    (effects (font (size 1 1) (thickness 0.1)) (justify mirror))
+  )
   (gr_line (start 164 86) (end 135 86) (layer Edge.Cuts) (width 0.15))
   (gr_line (start 135 40) (end 164 40) (layer Edge.Cuts) (width 0.15))
   (gr_line (start 135 86) (end 135 40) (layer Edge.Cuts) (width 0.2))
   (gr_line (start 164 86) (end 164 40) (layer Edge.Cuts) (width 0.15))
-  (via (at 143.125001 66.274999) (size 0.8) (drill 0.4) (layers F.Cu B.Cu) (net 9))
   (segment (start 141.505001 74.095001) (end 141.179999 73.769999) (width 0.25) (layer F.Cu) (net 4))
   (segment (start 141.505001 75.890003) (end 141.505001 74.095001) (width 0.25) (layer F.Cu) (net 4))
@@
   (segment (start 138.639999 69.530001) (end 137.79 70.38) (width 0.25) (layer F.Cu) (net 7))
   (segment (start 141.505001 68.994999) (end 141.484999 69.015001) (width 0.25) (layer F.Cu) (net 7))
+  (via (at 143.125001 66.274999) (size 0.8) (drill 0.4) (layers F.Cu B.Cu) (net 9))
   (segment (start 154.665001 56.374999) (end 143.125001 56.374999) (width 0.25) (layer F.Cu) (net 9))
   (segment (start 161.54 49.5) (end 154.665001 56.374999) (width 0.25) (layer F.Cu) (net 9))
