File: hardware/Expansion Boards/Blink/Blink.kicad_pcb (KiCad board)
At the start: 2 copper layers, 29 x 46 mm, 13 parts, among them J1 Daughter Board Connector

Commit message: New Blink Expansion Board
Signed-off-by: John Jacques <eruditelite@gmail.com>
Parts:
- D1, D2, D3, D4, D5, D6: moved to F.Cu
- J1, R1, R2, R3, R4, R5, R6: moved to B.Cu
- moved D4 302.6 mm to (317.6, 307.3), turned to 180 degrees
- moved J1 298.9 mm to (294.7, 334.0), turned to 0 degrees
- moved D5 293.9 mm to (310.3, 316.5), turned to 180 degrees
- moved D1 289.3 mm to (279.5, 308.0), turned to 180 degrees
- moved D2 288.1 mm to (280.2, 321.2), turned to 180 degrees
- moved D3 284.2 mm to (279.5, 334.2), turned to 180 degrees
- moved D6 272.5 mm to (311.5, 307.3), turned to 180 degrees
- moved R4 261.4 mm to (296.2, 262.4), turned to 180 degrees
- moved R1 260.0 mm to (296.2, 254.3), turned to 180 degrees
- moved R2 250.8 mm to (296.2, 258.3), turned to 180 degrees
- moved R6 238.4 mm to (296.2, 266.4), turned to 180 degrees
- moved R5 237.8 mm to (282.9, 258.3), turned to 180 degrees
- moved R3 226.3 mm to (282.9, 254.3), turned to 180 degrees
Connections:
- D4 pad 2: /ATtiny85_PB0 -> /ATtiny85_PB1
- D5 pad 2: /ATtiny85_PB1 -> /ATtiny85_PB3
- D6 pad 2: /ATtiny85_PB2 -> /ATtiny85_PB4
Routing:
- net /ATtiny85_PB1: track 77.0 -> 0.00 mm
- net /ATtiny85_PB2: track 44.1 -> 0.00 mm
- net /ATtiny85_PB0: track 37.1 -> 0.00 mm, vias 1 -> 0
- net /ATtiny84_PB0: track 30.2 -> 0.00 mm
- net /ATtiny84_PB1: track 18.5 -> 0.00 mm
- net /ATtiny84_PB2: track 17.6 -> 0.00 mm
- net Net-(D6-Pad1): track 9.62 -> 0.00 mm
- net Net-(D3-Pad1): track 9.62 -> 0.00 mm
- net Net-(D5-Pad1): track 9.62 -> 0.00 mm
- net Net-(D4-Pad1): track 9.62 -> 0.00 mm
- net Net-(D1-Pad1): track 9.62 -> 0.00 mm
- net Net-(D2-Pad1): track 9.12 -> 0.00 mm
- removed copper zone on B.Cu, net GND
Other:
- board size 29 x 46 mm -> 51 x 46 mm
- board text removed: "BLIINK"
- board text removed: "PB0@84"
- board text removed: "PB0@85"
- board text removed: "PB1@84"
- board text removed: "PB1@85"
- board text removed: "PB2@84"
- board text removed: "PB2@85"
