File: hardware/Expansion Boards/Expansion Board Template/Expansion Board Template.sch (KiCad schematic (older format))
At the start: 1 part, among them J1 Daughter Board Connector

Commit message: The New (v2) Board
Signed-off-by: John Jacques <eruditelite@gmail.com>
Parts:
- added MK1, MK2, MK3, MK4: M2.5, MountingHole:MountingHole_2.7mm_M2.5, symbol Expansion-Board-Template-rescue:Mounting_Hole-Mechanical
- J1: value Daughter Board Connector -> Conn_02x10_Odd_Even
Connections:
- net labels removed: +3.3V, +5V, ATtiny84_PA0, ATtiny84_PA1, ATtiny84_PA2, ATtiny84_PA3, ATtiny84_PA4, ATtiny84_PA5, ATtiny84_PA6, ATtiny84_PA7, ATtiny84_PB0, ATtiny84_PB1, ATtiny84_PB2, ATtiny85_PB0, ATtiny85_PB1, ATtiny85_PB2, ATtiny85_PB3, ATtiny85_PB4, GND
- wire segments 24 -> 0
Other:
- note added: "ID_SD and ID_SC PINS:\nThese pins are reserved for HAT ID EEPROM.\n\nAt boot time this I2C interface will be\ninterrogated to look for an EEPROM\nthat identifes the attached board and\nallows automagic setup of the GPIOs\n(and optionally, Linux drivers).\n\nDO NOT USE these pins for anything other\nthan attaching an I2C ID EEPROM. Leave\nunconnected if ID EEPROM not required."
- note added: "Mounting Holes"
Changed lines of the file:
@@
 EESchema Schematic File Version 4
-LIBS:Blink-cache
-EELAYER 26 0
+LIBS:Expansion Board Template-cache
+EELAYER 29 0
 EELAYER END
 $Descr A4 11693 8268
@@
 Sheet 1 1
 Title ""
-Date ""
+Date "15 nov 2012"
 Rev ""
 Comp ""
@@
 Comment4 ""
 $EndDescr
+Text Notes 650  7600 0    50   ~ 0
+ID_SD and ID_SC PINS:\nThese pins are reserved for HAT ID EEPROM.\n\nAt boot time this I2C interface will be\ninterrogated to look for an EEPROM\nthat identifes the attached board and\nallows automagic setup of the GPIOs\n(and optionally, Linux drivers).\n\nDO NOT USE these pins for anything other\nthan attaching an I2C ID EEPROM. Leave\nunconnected if ID EEPROM not required.
+$Comp
+L Expansion-Board-Template-rescue:Mounting_Hole-Mechanical MK1
+U 1 1 5834FB2E
+P 3000 7200
+F 0 "MK1" H 3100 7246 50  0000 L CNN
+F 1 "M2.5" H 3100 7155 50  0000 L CNN
+F 2 "MountingHole:MountingHole_2.7mm_M2.5" H 3000 7200 60  0001 C CNN
+F 3 "" H 3000 7200 60  0001 C CNN
+	1    3000 7200
+	1    0    0    -1
+$EndComp
+$Comp
+L Expansion-Board-Template-rescue:Mounting_Hole-Mechanical MK3
+U 1 1 5834FBEF
+P 3450 7200
+F 0 "MK3" H 3550 7246 50  0000 L CNN
+F 1 "M2.5" H 3550 7155 50  0000 L CNN
+F 2 "MountingHole:MountingHole_2.7mm_M2.5" H 3450 7200 60  0001 C CNN
+F 3 "" H 3450 7200 60  0001 C CNN
+	1    3450 7200
+	1    0    0    -1
+$EndComp
+$Comp
+L Expansion-Board-Template-rescue:Mounting_Hole-Mechanical MK2
+U 1 1 5834FC19
+P 3000 7400
+F 0 "MK2" H 3100 7446 50  0000 L CNN
+F 1 "M2.5" H 3100 7355 50  0000 L CNN
+F 2 "MountingHole:MountingHole_2.7mm_M2.5" H 3000 7400 60  0001 C CNN
+F 3 "" H 3000 7400 60  0001 C CNN
+	1    3000 7400
+	1    0    0    -1
+$EndComp
+$Comp
+L Expansion-Board-Template-rescue:Mounting_Hole-Mechanical MK4
+U 1 1 5834FC4F
+P 3450 7400
+F 0 "MK4" H 3550 7446 50  0000 L CNN
+F 1 "M2.5" H 3550 7355 50  0000 L CNN
+F 2 "MountingHole:MountingHole_2.7mm_M2.5" H 3450 7400 60  0001 C CNN
+F 3 "" H 3450 7400 60  0001 C CNN
+	1    3450 7400
+	1    0    0    -1
+$EndComp
+Text Notes 3000 7050 0    50   ~ 0
+Mounting Holes
 $Comp
 L Connector_Generic:Conn_02x10_Odd_Even J1
-U 1 1 5CD86BAC
-P 2550 3000
-F 0 "J1" H 2600 2350 50  0000 C CNN
-F 1 "Daughter Board Connector" H 2100 2100 50  0000 C CNN
-F 2 "Connector_PinHeader_2.54mm:PinHeader_2x10_P2.54mm_Vertical" H 2550 3000 50  0001 C CNN
-F 3 "~" H 2550 3000 50  0001 C CNN
-	1    2550 3000
+U 1 1 5CB1F643
+P 5700 3500
+F 0 "J1" H 5750 4117 50  0000 C CNN
+F 1 "Conn_02x10_Odd_Even" H 6450 4500 50  0000 C CNN
+F 2 "Connector_PinHeader_2.54mm:PinHeader_2x10_P2.54mm_Vertical" H 5850 2600 50  0000 C CNN
+F 3 "~" H 5700 3500 50  0001 C CNN
+	1    5700 3500
 	1    0    0    -1
 $EndComp
-Text Label 1650 2600 0    50   ~ 0
-ATtiny84_PA6
-Wire Wire Line
-	1650 2600 2350 2600
-Text Label 1650 2700 0    50   ~ 0
-ATtiny84_PA7
-Wire Wire Line
-	1650 2700 2350 2700
-Text Label 1650 2800 0    50   ~ 0
-ATtiny84_PB2
-Text Label 1650 2900 0    50   ~ 0
-ATtiny84_PA5
-Text Label 1650 3000 0    50   ~ 0
-ATtiny84_PA4
-Text Label 1650 3100 0    50   ~ 0
-ATtiny84_PA3
-Text Label 1650 3200 0    50   ~ 0
-ATtiny84_PA2
-Text Label 1650 3300 0    50   ~ 0
-ATtiny84_PA1
-Text Label 1650 3400 0    50   ~ 0
-ATtiny84_PA0
-Wire Wire Line
-	1650 2800 2350 2800
-Wire Wire Line
-	1650 2900 2350 2900
-Wire Wire Line
-	1650 3000 2350 3000
-Wire Wire Line
-	1650 3100 2350 3100
-Wire Wire Line
-	1650 3200 2350 3200
-Wire Wire Line
-	1650 3300 2350 3300
-Wire Wire Line
-	1650 3400 2350 3400
-Wire Wire Line
-	2350 3500 2300 3500
-Wire Wire Line
-	2300 3500 2300 2450
-$Comp
-L power:+5V #PWR0101
-U 1 1 5CD8E5C1
-P 2300 2450
-F 0 "#PWR0101" H 2300 2300 50  0001 C CNN
-F 1 "+5V" H 2315 2623 50  0000 C CNN
-F 2 "" H 2300 2450 50  0001 C CNN
-F 3 "" H 2300 2450 50  0001 C CNN
-	1    2300 2450
-	1    0    0    -1
-$EndComp
-Wire Wire Line
-	2850 2600 2950 2600
-Wire Wire Line
-	2950 2600 2950 2700
-Wire Wire Line
-	2850 2700 2950 2700
-Connection ~ 2950 2700
-Wire Wire Line
-	2950 2700 2950 3750
-$Comp
-L power:GND #PWR0102
-U 1 1 5CD8E7FF
-P 2950 3750
-F 0 "#PWR0102" H 2950 3500 50  0001 C CNN
-F 1 "GND" H 2955 3577 50  0000 C CNN
-F 2 "" H 2950 3750 50  0001 C CNN
-F 3 "" H 2950 3750 50  0001 C CNN
-	1    2950 3750
-	1    0    0    -1
-$EndComp
-Text Label 3600 2800 2    50   ~ 0
-ATtiny84_PB1
-Wire Wire Line
-	2850 3500 3050 3500
-Wire Wire Line
-	3050 3500 3050 2450
-$Comp
-L power:+3.3V #PWR0103
-U 1 1 5CD8E9EA
-P 3050 2450
-F 0 "#PWR0103" H 3050 2300 50  0001 C CNN
-F 1 "+3.3V" H 3065 2623 50  0000 C CNN
-F 2 "" H 3050 2450 50  0001 C CNN
-F 3 "" H 3050 2450 50  0001 C CNN
-	1    3050 2450
-	1    0    0    -1
-$EndComp
-Text Label 3600 2900 2    50   ~ 0
-ATtiny84_PB0
-Text Label 3600 3000 2    50   ~ 0
-ATtiny85_PB0
-Text Label 3600 3100 2    50   ~ 0
-ATtiny85_PB1
-Text Label 3600 3200 2    50   ~ 0
-ATtiny85_PB2
-Text Label 3600 3300 2    50   ~ 0
-ATtiny85_PB4
-Text Label 3600 3400 2    50   ~ 0
-ATtiny85_PB3
-Wire Wire Line
-	2850 2800 3600 2800
-Wire Wire Line
-	2850 2900 3600 2900
-Wire Wire Line
-	2850 3000 3600 3000
-Wire Wire Line
-	2850 3100 3600 3100
-Wire Wire Line
-	2850 3200 3600 3200
-Wire Wire Line
-	2850 3300 3600 3300
-Wire Wire Line
-	2850 3400 3600 3400
 $EndSCHEMATC
